Commit message: make xacro files. Confusing asf. Now it does not work. cant find common_properties.xacro why????? it is literally there

File: tb3_description/urdf/common_properties.xacro (robot description, xacro)
@@ -1,28 +1,20 @@
 <?xml version="1.0"?>
 <robot xmlns:xacro="http://ros.org/wiki/xacro">
-  <!--
-    These properties must be observed by any machine
-    that wants to be defined as a turtlebot. Refer
-    to the REP for more details.
-    http://www.ros.org/reps/rep-0119.html
-   -->
-  <!--
-   ======================================================================
-   - REP 119 : Rgb camera link relative to the Base link
-   ======================================================================
-     Base link is currently defined as the rotational centre on the bottom
-     of the base mould. For both create and kobuki this is actually exactly
-     the same 3d world point.
-     This may cause an issue with a base with much different floor clearance.
-     Should we be using base_footprint for this specification instead?
-     Note: REP needs to be updated with the information below
-     (currently in development and awaiting feedback)
-   -->
-  <xacro:property name="M_PI" value="3.14159265359"/>
-  <xacro:property name="cam_px" value="-0.087" />
-<!--  <xacro:property name="cam_py" value="-0.0125" /> Y varies for different configurations. get sets in sensors_urdf -->
-  <xacro:property name="cam_pz" value="0.2870" />
-	<xacro:property name="cam_or" value="0" />
-	<xacro:property name="cam_op" value="0" />
-	<xacro:property name="cam_oy" value="0" />
+  <!-- Common inertial properties -->
+  <xacro:property name="default_mass" value="0.1"/>
+  <xacro:property name="default_inertia" value="0.001"/>
+  <!-- Default material definitions -->
+  <material name="light_black">
+    <color rgba="0.2 0.2 0.2 1.0"/>
+  </material>
+  <material name="dark">
+    <color rgba="0.1 0.1 0.1 1.0"/>
+  </material>
+  <material name="orange">
+    <color rgba="1.0 0.5 0.0 1.0"/>
+  </material>
+  <!-- Common dimensions -->
+  <xacro:property name="wheel_radius" value="0.033"/>
+  <xacro:property name="wheel_width" value="0.018"/>
+  <xacro:property name="caster_radius" value="0.005"/>
 </robot>
